File: PCB/MacroPad.kicad_sch (KiCad schematic)
At the start: 11 parts, among them SW1 SW_Push, SW2 SW_Push, SW3 SW_Push, SW4 SW_Push, SW5 SW_Push, SW6 SW_Push, U1 XIAO-RP2040-DIP

Commit message: fixed wrong footprint for SK6812MINI-E
Parts:
- D1: value SK6812MINI -> MINI-E:SK6812MINI-E_fixed; footprint LED_SMD:LED_SK6812MINI_PLCC4_3.5x3.5mm_P1.75mm -> MINI-E:SK6812MINI-E_fixed
- D2, D3, D4: footprint LED_SMD:LED_SK6812MINI_PLCC4_3.5x3.5mm_P1.75mm -> MINI-E:SK6812MINI-E_fixed
Changed lines of the file:
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@@
 			)
 		)
-		(property "Value" "SK6812MINI"
+		(property "Value" "MINI-E:SK6812MINI-E_fixed"
 			(at 195.58 44.5202 0)
 			(effects
@@
 			)
 		)
-		(property "Footprint" "LED_SMD:LED_SK6812MINI_PLCC4_3.5x3.5mm_P1.75mm"
+		(property "Footprint" "MINI-E:SK6812MINI-E_fixed"
 			(at 207.01 33.02 0)
 			(effects
@@
 			)
 		)
-		(property "Footprint" "LED_SMD:LED_SK6812MINI_PLCC4_3.5x3.5mm_P1.75mm"
+		(property "Footprint" "MINI-E:SK6812MINI-E_fixed"
 			(at 156.21 33.02 0)
 			(effects
@@
 			)
 		)
-		(property "Footprint" "LED_SMD:LED_SK6812MINI_PLCC4_3.5x3.5mm_P1.75mm"
+		(property "Footprint" "MINI-E:SK6812MINI-E_fixed"
 			(at 134.62 33.02 0)
 			(effects
@@
 			)
 		)
-		(property "Footprint" "LED_SMD:LED_SK6812MINI_PLCC4_3.5x3.5mm_P1.75mm"
+		(property "Footprint" "MINI-E:SK6812MINI-E_fixed"
 			(at 182.88 33.02 0)
 			(effects
